File: MacVRAMSIMM.kicad_pcb (KiCad board)
At the start: 4 copper layers, 102.9 x 20.3 mm, 17 parts, among them J1 VRAM, U1 42C8255, U2 42C8255

Commit message: Fabbed
Parts:
- renumbered C1 to C5, C1 to C6
Connections:
- net Net-(J1-Pad23) renamed /L~OE~2
- net Net-(J1-Pad28) renamed /L~WE~2
- net Net-(J1-Pad57) renamed /U~OE~2
- net Net-(J1-Pad62) renamed /U~WE~2
Routing:
- net GND: track 50.8 -> 52.9 mm, vias 118 -> 120
