File: MacVRAMSIMM.sch (KiCad schematic (older format))
At the start: 15 parts, among them J1 VRAM, U1 42C8255, U2 42C8255

Commit message: Fabbed
Parts:
- added C5, C6: 2u2, stdpads:C_0805, symbol Device:C_Small
Connections:
- net +5V: now also C5.1, C6.1
- net GND: now also C5.2, C6.2
- net UL~OE~2 renamed U~OE~2
Other:
- moved on the sheet: C1, C2, C3, C4, FID1, FID2, FID3, FID4, H1, H2, H3, H4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
